File: microphone_array_v2.kicad_pcb (KiCad board)
At the start: 4 copper layers, 120 x 120 mm, 124 parts, among them J1 RPi_P1_26, J2 Tang_Nano_9K, J3 Tang_Nano_9K, U1 LP5907MFX-3.3, U2 SN74LVC244A, U3 USBLC6-4SC6, U4 USBLC6-4SC6, X1 24.576MHz

Commit message: Build board
Routing:
- net +3V3A: track 411.7 -> 434.7 mm, vias 22 -> 28
- net PDM_CLK_B3: track 85.3 -> 108.1 mm
- net GND: track 111.3 -> 133.7 mm
- net HOST_RESET_N: track 22.5 -> 43.6 mm, vias 4 -> 2
- net PDM_CLK_B4: track 85.6 -> 105.5 mm
- net PDM_CLK_B0: track 89.9 -> 107.2 mm
- net PDM_CLK_B2: track 90.6 -> 104.8 mm
- net PDM_CLK_B1: track 90.2 -> 103.7 mm
- net PDM_CLK_IN: track 25.7 -> 38.0 mm, vias 3 -> 0
- net PI_IRQ: track 19.8 -> 31.4 mm
- net PI_STATUS: track 16.6 -> 27.3 mm, vias 3 -> 2
- net PDM_CLK_FPGA: track 19.2 -> 29.6 mm, vias 2 -> 0
- net PI_MOSI: track 30.5 -> 20.8 mm
- net PI_MISO: track 40.5 -> 50.2 mm, vias 3 -> 2
- net PDM_D6: track 61.7 -> 70.3 mm
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Other:
- board text added: "+3V3A"
- board text added: "+3V3_CLK"
- board text added: "+5V"
- board text added: "GND"
- board text added: "HOST_STATUS"
- board text added: "PDM_D0"
- board text added: "PDM_D1"
- board text added: "PDM_D2"
- board text added: "PDM_D3"
- board text added: "PDM_D4"
- board text added: "PDM_D5"
- board text added: "PDM_D6"
- board text added: "PDM_D7"

Commit message: New board rev
Parts:
- removed H1, H2, H3, H4: M3, MountingHole:MountingHole_3.2mm_M3
- J1: footprint Connector_PinHeader_2.54mm:PinHeader_2x13_P2.54mm_Vertical -> Connector_PinSocket_2.54mm:PinSocket_2x13_P2.54mm_Vertical
- moved J1 2.54 mm to (165.2, 179.2)
Connections:
- U3 pad 1: PI_RESET_N -> PI_SCLK
- U3 pad 3: PI_SCLK -> PI_RESET_N
- U3 pad 4: PI_CS_N -> PI_MISO
- U3 pad 6: PI_MISO -> PI_CS_N
- U4 pad 1: PI_IRQ -> PI_MOSI
- U4 pad 3: PI_MOSI -> PI_IRQ
- U4 pad 4: PI_STATUS -> PI_SYNC
- U4 pad 6: PI_SYNC -> PI_STATUS
Routing:
- net PI_MISO: track 50.2 -> 11.9 mm, vias 2 -> 1
- net HOST_RESET_N: track 43.6 -> 18.8 mm, vias 2 -> 3
- net PI_IRQ: track 31.4 -> 49.1 mm, vias 2 -> 3
- net PI_CS_N: track 12.1 -> 26.2 mm
- net PI_SCLK: track 22.2 -> 10.5 mm, vias 1 -> 2
- net PI_MOSI: track 20.8 -> 11.9 mm, vias 2 -> 1
- net PI_5V: track 50.6 -> 58.7 mm
- net PI_RESET_N: track 9.91 -> 15.9 mm, vias 2 -> 0
- net PI_SYNC: track 14.5 -> 20.5 mm, vias 2 -> 0
- net PI_STATUS: track 27.3 -> 22.7 mm, vias 2 -> 3
- net +3V3_CLK: track 63.3 -> 62.8 mm
- net TANG_3V3: track 39.5 -> 39.6 mm, vias 7 -> 3
